Commit message: Added STL to Mesh

File: src/crustcrawler_description/urdf/first.xacro (robot description, xacro)
@@ -17,5 +17,5 @@
     <visual>
       <geometry>
-        <box size="${LinkWidth} ${LinkWidth} ${L1}"/>
+        <mesh filename="package://crustcrawler_description/meshes/BaseLink.STL"/>
       </geometry>
       <origin rpy="0 0 0" xyz="0 0 ${-L1+L1/2}"/>

Commit message: HotFix

File: src/crustcrawler_description/urdf/first.xacro (robot description, xacro)
@@ -17,5 +17,5 @@
     <visual>
       <geometry>
-        <mesh filename="package://crustcrawler_description/meshes/BaseLink.STL"/>
+        <box size="${L2} ${LinkWidth} ${LinkWidth}"/>
       </geometry>
       <origin rpy="0 0 0" xyz="0 0 ${-L1+L1/2}"/>
