Commit message: more stuff done

File: src/crustcrawler_description/urdf/crustcrawler_old.xacro (robot description, xacro)
@@ -69,5 +69,5 @@
       <origin xyz="0 0 ${L1/2}" rpy="0 0 0"/>
       <geometry>
-        <box size="${LinkWidth} ${LinkWidth} ${L1}"/>
+	<box size="${LinkWidth} ${LinkWidth} ${L1}"/>
       </geometry>
     </collision>
@@ -75,5 +75,5 @@
       <origin xyz="0 0 ${L1/2}" rpy="0 0 0"/>
       <geometry>
-        <mesh filename="package://crustcrawler_description/meshes/Link1.STL"/>
+	<box size="${LinkWidth} ${LinkWidth} ${L1}"/>
       </geometry>
     </visual>
