Commit message: Working Script.

File: src/crustcrawler_description/urdf/crustcrawler.xacro (robot description, xacro)
@@ -1,9 +1,16 @@
 <?xml version="1.0"?>
 <robot xmlns:xacro="http://www.ros.org/wiki/xacro" name="CrustCrawler">
-  <xacro:property name="pi" value="3.1415" />
+  <xacro:property name="M_pi" value="3.1415" />
   <xacro:property name="LinkWidth" value="0.01" />
   <xacro:property name="L1" value="0.055" />
   <xacro:property name="L2" value="0.22" />
   <xacro:property name="Lcp" value="0.15" />
+  <xacro:property name="Lc" value="0.05875" />
+  <xacro:property name="Lc2" value="0.17433" />
+  <xacro:property name="Lc3" value="0.12078" />
+  <xacro:property name="m1" value="0.22501148645" />
+  <xacro:property name="m2" value="0.21285774246" />
+  <xacro:property name="m3" value="0.28725035108" />
+  <xacro:property name="mp" value="0.0" />
   <link name="base_link">
     <visual>
@@ -17,8 +24,19 @@
     <visual>
       <geometry>
+        <box size="${LinkWidth} ${LinkWidth} ${L2}"/>
+      </geometry>
+      <origin rpy="0 0 0" xyz="0 0 ${-L1+L1/2}"/>
+    </visual>
+    <collision>
+      <geometry>
         <box size="${L2} ${LinkWidth} ${LinkWidth}"/>
       </geometry>
       <origin rpy="0 0 0" xyz="0 0 ${-L1+L1/2}"/>
-    </visual>
+    </collision>
+    <inertial>
+      <mass value="${m1}"/>
+      <origin rpy="0 0 0" xyz="0 0 ${-L1+Lc}"/>
+      <inertia ixx="1.0" ixy="0.0" ixz="0.0" iyy="1.0" iyz="0.0" izz="1.0"/>
+    </inertial>
   </link>
   <link name="link2">
@@ -29,4 +47,14 @@
       <origin rpy="0 0 0" xyz="${L2/2} 0 0"/>
     </visual>
+    <collision>
+      <geometry>
+        <box size="${L2} ${LinkWidth} ${LinkWidth}"/>
+      </geometry>
+      <origin rpy="0 0 0" xyz="${L2/2} 0 0"/>
+    </collision>
+    <inertial>
+      <mass value="${m2}"/>
+      <inertia ixx="1.0" ixy="0.0" ixz="0.0" iyy="1.0" iyz="0.0" izz="1.0"/>
+    </inertial>
   </link>
   <link name="link3">
@@ -37,8 +65,30 @@
       <origin rpy="0 0 0" xyz="${Lcp/2} 0 0"/>
     </visual>
+    <collision>
+      <geometry>
+        <box size="${Lcp} ${LinkWidth} ${LinkWidth}"/>
+      </geometry>
+      <origin rpy="0 0 0" xyz="${Lcp/2} 0 0"/>
+    </collision>
+    <inertial>
+      <mass value="${m3}"/>
+      <inertia ixx="1.0" ixy="0.0" ixz="0.0" iyy="1.0" iyz="0.0" izz="1.0"/>
+    </inertial>
+  </link>
+  <link name="link4">
+    <visual>
+      <geometry>
+        <box size="${LinkWidth} ${LinkWidth} ${LinkWidth}"/>
+      </geometry>
+      <origin rpy="0 0 0" xyz="0 0 0"/>
+    </visual>
+    <inertial>
+      <mass value="${mp}"/>
+      <inertia ixx="0.0" ixy="0.0" ixz="0.0" iyy="0.0" iyz="0.0" izz="0.0"/>
+    </inertial>
   </link>
   <joint name="FirstJoint" type="revolute">
     <axis xyz="0 0 1"/>
-    <limit effort="1000.0" lower="0.0" upper="${pi*2}" velocity="0.5"/>
+    <limit effort="1000.0" lower="0.0" upper="${M_pi*2}" velocity="0.5"/>
     <parent link="base_link"/>
     <child link="link1"/>
@@ -47,8 +97,8 @@
   <joint name="SecondJoint" type="revolute">
     <axis xyz="0 0 1"/>
-    <limit effort="1000.0" lower="-0.3" upper="${pi}" velocity="0.5"/>
+    <limit effort="1000.0" lower="-0.3" upper="${M_pi}" velocity="0.5"/>
     <parent link="link1"/>
     <child link="link2"/>
-    <origin xyz="0 0 0" rpy="${pi/2} 0 0"/>
+    <origin xyz="0 0 0" rpy="${M_pi/2} 0 0"/>
   </joint>
   <joint name="ThirdJoint" type="revolute">
@@ -59,3 +109,8 @@
     <origin xyz="${L2} 0 0" rpy="0 0 0"/>
   </joint>
+  <joint name="PayloadJoint" type="fixed">
+    <parent link="link3"/>
+    <child link="link4"/>
+    <origin xyz="${Lcp} 0 0" rpy="0 0 0"/>
+  </joint>
 </robot>

Commit message: Bug Fix

File: src/crustcrawler_description/urdf/crustcrawler.xacro (robot description, xacro)
@@ -24,5 +24,5 @@
     <visual>
       <geometry>
-        <box size="${LinkWidth} ${LinkWidth} ${L2}"/>
+        <box size="${LinkWidth} ${LinkWidth} ${L1}"/>
       </geometry>
       <origin rpy="0 0 0" xyz="0 0 ${-L1+L1/2}"/>

Commit message: modeling close to done, adjust gripper/ physics

File: src/crustcrawler_description/urdf/crustcrawler.xacro (robot description, xacro)
@@ -4,5 +4,5 @@
   <xacro:property name="LinkWidth" value="0.01" />
   <xacro:property name="offset" value="0.0" />
-  <xacro:property name="L0" value="0.01" />
+  <xacro:property name="L0" value="0.0" />
   <xacro:property name="L1" value="0.055" />
   <xacro:property name="L2" value="0.22" />
@@ -23,5 +23,5 @@
   <link name="base">
     <collision>
-      <origin xyz="0 0 ${L0/2}" rpy="0 0 0"/>
+      <origin xyz="0 0 0" rpy="0 0 0"/>
       <geometry>
 	<box size="${LinkWidth} ${LinkWidth} ${L0}"/>
@@ -29,12 +29,12 @@
     </collision>
     <visual>
-      <origin xyz="0 0 ${L0/2}" rpy="0 0 0"/>
-      <geometry>
-	<box size="${LinkWidth} ${LinkWidth} ${L0}"/>
+      <origin xyz="0 0 ${-L1/2}" rpy="0 0 0"/>
+      <geometry>
+         <mesh filename="package://crustcrawler_description/meshes/Base.STL"/>           <!-- <box size="${LinkWidth} ${LinkWidth} ${L0}"/> -->
   <cylinder length="0.1" radius="0.1"/>
       </geometry>
     </visual>
     <inertial>
-      <origin xyz="0 0 ${L0/2}" rpy="0 0 0"/>
+      <origin xyz="0 0 0" rpy="0 0 0"/>
       <mass value="${m1}"/>
       <inertia
@@ -51,5 +51,5 @@
     <origin xyz="0 0 ${L0}" rpy= "0 0 0"/>
   </joint>
-  <!-- Turntable -->
+  <!-- Turntable
   <joint name="turntable" type="fixed">
     <parent link="base"/>
@@ -64,8 +64,9 @@
     </visual>
   </link>
+  -->
   <!-- link 1 -->
   <link name="link1">
     <collision>
-      <origin xyz="0 0 ${L1/2}" rpy="0 0 0"/>
+      <origin xyz="0 0 0" rpy="0 0 0"/>
       <geometry>
         <box size="${LinkWidth} ${LinkWidth} ${L1}"/>
@@ -73,5 +74,5 @@
     </collision>
     <visual>
-      <origin xyz="0 0 ${L1/2}" rpy="0 0 0"/>
+      <origin xyz="0 0 ${-L1/2}" rpy="0 0 0"/>
       <geometry>
         <mesh filename="package://crustcrawler_description/meshes/Link1.STL"/>
@@ -103,7 +104,7 @@
     </collision>
     <visual>
-      <origin xyz="${L2/2} 0 ${offset}" rpy="0 0 0"/>
-      <geometry>
-	<box size="${L2} ${LinkWidth} ${LinkWidth}"/>
+      <origin xyz="0 0 0.002" rpy="0 ${M_pi/2} 0"/>
+      <geometry>
+	       <mesh filename="package://crustcrawler_description/meshes/Link2.STL"/> <!--<box size="${L2} ${LinkWidth} ${LinkWidth}"/>-->
       </geometry>
     </visual>
@@ -133,7 +134,7 @@
     </collision>
     <visual>
-      <origin xyz="${L3/2} 0 0" rpy="0 0 0"/>
-      <geometry>
-  <box size="${L3} ${LinkWidth} ${LinkWidth} "/>
+      <origin xyz="0 0 0" rpy="0 ${M_pi/2} 0"/>
+      <geometry>
+        <mesh filename="package://crustcrawler_description/meshes/Link3.STL"/> <!--<box size="${L3} ${LinkWidth} ${LinkWidth} "/> -->
       </geometry>
     </visual>
@@ -147,3 +148,63 @@
     </inertial>
   </link>
+  <joint name="joint_4" type="revolute">
+    <axis xyz="0 0 1"/>
+    <limit effort="1000.0" lower="${-M_pi*3/4}" upper="${M_pi*3/4}" velocity="0.5"/>
+    <parent link="link3"/>
+    <child link="gripper_left"/>
+    <origin xyz="${L3 - 0.003} 0 0.016" rpy="${-M_pi/2} 0 0"/>
+  </joint>
+  <joint name="joint_5" type="revolute">
+    <axis xyz="0 0 1"/>
+    <limit effort="1000.0" lower="${-M_pi*3/4}" upper="${M_pi*3/4}" velocity="0.5"/>
+    <parent link="link3"/>
+    <child link="gripper_right"/>
+    <origin xyz="${L3 - 0.003} 0 -0.016" rpy="${-M_pi/2} 0 0"/>
+  </joint> -->
+  <!-- left gripper -->
+  <link name="gripper_left">
+    <collision>
+      <origin xyz="0 0 0" rpy="0 0 0.1"/>
+      <geometry>
+  <box size=" ${LinkWidth} ${LinkWidth} ${LinkWidth}"/>
+      </geometry>
+    </collision>
+    <visual>
+      <origin xyz="${-L3 + 0.001} 0.016   0" rpy="${M_pi/2} 0 ${M_pi/2}"/>
+      <geometry>
+        <mesh filename="package://crustcrawler_description/meshes/Grip.STL"/>
+      </geometry>
+    </visual>
+    <inertial>
+      <origin xyz="0 0 0 " rpy="0 0 0"/>
+      <mass value="0.001"/>
+      <inertia
+    ixx="1.0" ixy="0.0" ixz="0.0"
+    iyy="1.0" iyz="0.0"
+    izz="1.0"/>
+    </inertial>
+  </link>
+  <!-- right gripper -->
+  <link name="gripper_right">
+    <collision>
+      <origin xyz="0 0 0" rpy="0 0 0"/>
+      <geometry>
+  <box size=" ${LinkWidth} ${LinkWidth} ${LinkWidth}"/>
+      </geometry>
+    </collision>
+    <visual>
+      <origin xyz="${-L3 + 0.001} -0.016  0" rpy="${-M_pi/2} 0 ${-M_pi/2}"/>
+      <geometry>
+        <mesh filename="package://crustcrawler_description/meshes/Grip.STL"/>
+      </geometry>
+    </visual>
+    <inertial>
+      <origin xyz="0 0 0 " rpy="0 0 0"/>
+      <mass value="0.001"/>
+      <inertia
+    ixx="1.0" ixy="0.0" ixz="0.0"
+    iyy="1.0" iyz="0.0"
+    izz="1.0"/>
+    </inertial>
+  </link>
 </robot>

Commit message: raised robot above ground

File: src/crustcrawler_description/urdf/crustcrawler.xacro (robot description, xacro)
@@ -20,4 +20,5 @@
     <parent link="world"/>
     <child link="base"/>
+    <origin xyz = "0 0 0.15" />
   </joint>
   <link name="base">

Commit message: added rviz launch options

File: src/crustcrawler_description/urdf/crustcrawler.xacro (robot description, xacro)
@@ -16,4 +16,11 @@
   <xacro:property name="m3" value="0.28725035108" />
   <xacro:property name="mp" value="0.0" />
+  <!-- Gazebo -->
+  <gazebo>
+    <plugin name="gazebo_ros_control" filename="libgazebo_ros_control.so">
+      <robotNamespace>/crustcrawler</robotNamespace>
+    </plugin>
+  </gazebo>
+  <!-- links, joints and transmissions -->
   <link name="world"/>
   <joint name="world_base" type="fixed">
@@ -45,5 +52,5 @@
     </inertial>
   </link>
-  <joint name="joint_1" type="revolute">
+  <joint name="joint1" type="revolute">
     <axis xyz="0 0 1"/>
     <limit effort="1000.0" lower="${-M_pi}" upper="${M_pi}" velocity="0.5"/>
@@ -52,18 +59,14 @@
     <origin xyz="0 0 ${L0}" rpy= "0 0 0"/>
   </joint>
-  <!-- Turntable
-  <joint name="turntable" type="fixed">
-    <parent link="base"/>
-    <child link="turntable"/>
-  </joint>
-  <link name="turntable">
-    <visual>
-      <origin xyz="0 0 0" rpy="0 0 0"/>
-      <geometry>
-  <cylinder length="0.01" radius="0.04"/>
-      </geometry>
-    </visual>
-  </link>
-  -->
+  <transmission name="tran1">
+    <type>transmission_interface/SimpleTransmission</type>
+    <joint name="joint1">
+      <hardwareInterface>EffortJointInterface</hardwareInterface>
+    </joint>
+    <actuator name="motor1">
+      <hardwareInterface>EffortJointInterface</hardwareInterface>
+      <mechanicalReduction>1</mechanicalReduction>
+    </actuator>
+  </transmission>
   <!-- link 1 -->
   <link name="link1">
@@ -89,5 +92,5 @@
     </inertial>
   </link>
-  <joint name="joint_2" type="revolute">
+  <joint name="joint2" type="revolute">
     <origin xyz="0 0 ${L1}" rpy="${M_pi / 2} 0 0"/>
     <axis xyz="0 0 1"/>
@@ -119,5 +122,5 @@
     </inertial>
   </link>
-  <joint name="joint_3" type="revolute">
+  <joint name="joint3" type="revolute">
     <axis xyz="0 0 1"/>
     <limit effort="1000.0" lower="${-M_pi*3/4}" upper="${M_pi*3/4}" velocity="0.5"/>
@@ -149,5 +152,5 @@
     </inertial>
   </link>
-  <joint name="joint_4" type="revolute">
+  <joint name="joint4" type="revolute">
     <axis xyz="0 0 1"/>
     <limit effort="1000.0" lower="${-M_pi*3/4}" upper="${M_pi*3/4}" velocity="0.5"/>
@@ -156,5 +159,5 @@
     <origin xyz="${L3 - 0.003} 0 0.016" rpy="${-M_pi/2} 0 0"/>
   </joint>
-  <joint name="joint_5" type="revolute">
+  <joint name="joint5" type="revolute">
     <axis xyz="0 0 1"/>
     <limit effort="1000.0" lower="${-M_pi*3/4}" upper="${M_pi*3/4}" velocity="0.5"/>

Commit message: added damping

File: src/crustcrawler_description/urdf/crustcrawler.xacro (robot description, xacro)
@@ -58,12 +58,13 @@
     <child link="link1"/>
     <origin xyz="0 0 ${L0}" rpy= "0 0 0"/>
+    <dynamics damping="1.0"/>
   </joint>
   <transmission name="tran1">
     <type>transmission_interface/SimpleTransmission</type>
     <joint name="joint1">
-      <hardwareInterface>EffortJointInterface</hardwareInterface>
+      <hardwareInterface>hardware_interface/EffortJointInterface</hardwareInterface>
     </joint>
     <actuator name="motor1">
-      <hardwareInterface>EffortJointInterface</hardwareInterface>
+      <hardwareInterface>hardware_interface/EffortJointInterface</hardwareInterface>
       <mechanicalReduction>1</mechanicalReduction>
     </actuator>
@@ -98,4 +99,5 @@
     <parent link="link1"/>
     <child link="link2"/>
+    <dynamics damping="1.0"/>
   </joint>
   <!-- link 2 -->
@@ -128,4 +130,5 @@
     <child link="link3"/>
     <origin xyz="${L2} 0 0" rpy="0 0 0"/>
+    <dynamics damping="1.0"/>
   </joint>
   <!-- link 3 -->
@@ -158,4 +161,5 @@
     <child link="gripper_left"/>
     <origin xyz="${L3 - 0.003} 0 0.016" rpy="${-M_pi/2} 0 0"/>
+    <dynamics damping="1.0"/>
   </joint>
   <joint name="joint5" type="revolute">
@@ -165,4 +169,5 @@
     <child link="gripper_right"/>
     <origin xyz="${L3 - 0.003} 0 -0.016" rpy="${-M_pi/2} 0 0"/>
+    <dynamics damping="1.0"/>
   </joint> -->
   <!-- left gripper -->

Commit message: SetForce and 30Hz update rate, dampning.

File: src/crustcrawler_description/urdf/crustcrawler.xacro (robot description, xacro)
@@ -60,5 +60,5 @@
     <child link="link1"/>
     <origin xyz="0 0 ${L0}" rpy= "0 0 0"/>
-    <dynamics damping="1.0"/>
+    <dynamics damping="0.7"/>
   </joint>
   <transmission name="tran1">
@@ -101,5 +101,5 @@
     <parent link="link1"/>
     <child link="link2"/>
-    <dynamics damping="1.0"/>
+    <dynamics damping="0.7"/>
   </joint>
   <!-- link 2 -->
@@ -132,5 +132,5 @@
     <child link="link3"/>
     <origin xyz="${L2} 0 0" rpy="0 0 0"/>
-    <dynamics damping="1.0"/>
+    <dynamics damping="0.7"/>
   </joint>
   <!-- link 3 -->
@@ -163,5 +163,5 @@
     <child link="gripper_left"/>
     <origin xyz="${L3 - 0.003} 0 0.016" rpy="${-M_pi/2} 0 0"/>
-    <dynamics damping="1.0"/>
+    <dynamics damping="0.7"/>
   </joint>
   <joint name="joint5" type="revolute">
@@ -171,5 +171,5 @@
     <child link="gripper_right"/>
     <origin xyz="${L3 - 0.003} 0 -0.016" rpy="${-M_pi/2} 0 0"/>
-    <dynamics damping="1.0"/>
+    <dynamics damping="0.7"/>
   </joint> -->
   <!-- left gripper -->

Commit message: collision box fix

File: src/crustcrawler_description/urdf/crustcrawler.xacro (robot description, xacro)
@@ -42,5 +42,5 @@
       <geometry>
          <mesh filename="package://crustcrawler_description/meshes/Base.STL"/>           <!-- <box size="${LinkWidth} ${LinkWidth} ${L0}"/> -->
-  <cylinder length="0.1" radius="0.1"/>
+         <!--cylinder length="0.1" radius="0.1"/-->
       </geometry>
     </visual>

Commit message: collision box fix

File: src/crustcrawler_description/urdf/crustcrawler.xacro (robot description, xacro)
@@ -2,7 +2,12 @@
 <robot name="CrustCrawler" xmlns:xacro="http://www.ros.org/wiki/xacro">
   <xacro:property name="M_pi" value="3.1415" />
-  <xacro:property name="LinkWidth" value="0.01" />
+  <xacro:property name="LinkWidth" value="0.025" />
+  <xacro:property name="LinkHeight" value="0.02" />
   <xacro:property name="offset" value="0.0" />
-  <xacro:property name="L0" value="0.0" />
+  <xacro:property name="MotorWidth" value="0.04" />
+  <xacro:property name="MotorLength" value="0.055" />
+  <xacro:property name="MotorOffset" value="0.04" />
+  <xacro:property name="BaseWidth" value="0.15" />
+  <xacro:property name="L0" value="0.01" />
   <xacro:property name="L1" value="0.055" />
   <xacro:property name="L2" value="0.22" />
@@ -12,4 +17,5 @@
   <xacro:property name="Lc2" value="0.17433" />
   <xacro:property name="Lc3" value="0.12078" />
+  <xacro:property name="d3" value="-0.003" />
   <xacro:property name="m1" value="0.22501148645" />
   <xacro:property name="m2" value="0.21285774246" />
@@ -24,4 +30,13 @@
     </plugin>
   </gazebo>
+  <gazebo reference="link1">
+    <selfCollide>true</selfCollide>
+  </gazebo>
+  <gazebo reference="link2">
+    <selfCollide>true</selfCollide>
+  </gazebo>
+  <gazebo reference="link3">
+    <selfCollide>true</selfCollide>
+  </gazebo>
   <!-- links, joints and transmissions -->
   <link name="world"/>
@@ -31,9 +46,10 @@
     <origin xyz = "0 0 0.15" />
   </joint>
+  <!-- base link -->
   <link name="base">
     <collision>
-      <origin xyz="0 0 0" rpy="0 0 0"/>
-      <geometry>
-	<box size="${LinkWidth} ${LinkWidth} ${L0}"/>
+      <origin xyz="0 0 -0.015" rpy="0 0 0"/>
+      <geometry>
+	       <box size="${BaseWidth} ${BaseWidth} 0.01"/>
       </geometry>
     </collision>
@@ -41,6 +57,5 @@
       <origin xyz="0 0 ${-L1/2}" rpy="0 0 0"/>
       <geometry>
-         <mesh filename="package://crustcrawler_description/meshes/Base.STL"/>           <!-- <box size="${LinkWidth} ${LinkWidth} ${L0}"/> -->
-         <!--cylinder length="0.1" radius="0.1"/-->
+         <mesh filename="package://crustcrawler_description/meshes/Base.STL"/>
       </geometry>
     </visual>
@@ -59,5 +74,5 @@
     <parent link="base"/>
     <child link="link1"/>
-    <origin xyz="0 0 ${L0}" rpy= "0 0 0"/>
+    <origin xyz="0 0 0" rpy= "0 0 0"/>
     <dynamics damping="0.7"/>
   </joint>
@@ -75,7 +90,7 @@
   <link name="link1">
     <collision>
-      <origin xyz="0 0 0" rpy="0 0 0"/>
-      <geometry>
-        <box size="${LinkWidth} ${LinkWidth} ${L1}"/>
+      <origin xyz="0 0 ${L1 / 2}" rpy="0 0 0"/>
+      <geometry>
+        <box size="${MotorWidth} ${MotorLength} ${L1*1.5}"/>
       </geometry>
     </collision>
@@ -90,7 +105,7 @@
       <mass value="${m1}"/>
       <inertia
-	  ixx="1.0" ixy="0.0" ixz="0.0"
-	  iyy="1.0" iyz="0.0"
-	  izz="1.0"/>
+    	  ixx="1.0" ixy="0.0" ixz="0.0"
+    	  iyy="1.0" iyz="0.0"
+    	  izz="1.0"/>
     </inertial>
   </link>
@@ -106,7 +121,13 @@
   <link name="link2">
     <collision>
-      <origin xyz="${L2/2} 0 0" rpy="0 0 0"/>
-      <geometry>
-	<box size="${L2} ${LinkWidth} ${LinkWidth}"/>
+      <origin xyz="${L2/2 - MotorOffset/2} 0 0" rpy="0 0 0"/>
+      <geometry>
+         <box size=" ${L2 - MotorOffset*3} ${LinkWidth} ${LinkHeight}"/>
+      </geometry>
+    </collision>
+    <collision>
+      <origin xyz = "${L2 - 0.015} 0 0" />
+      <geometry>
+         <box size=" ${0.05} ${MotorWidth} ${MotorLength}"/>
       </geometry>
     </collision>
@@ -137,7 +158,13 @@
   <link name="link3">
     <collision>
-      <origin xyz="${L3/2} 0 0" rpy="0 0 0"/>
-      <geometry>
-  <box size=" ${L3} ${LinkWidth} ${LinkWidth}"/>
+      <origin xyz="${L3/2} 0 ${d3}" rpy="0 0 0"/>
+      <geometry>
+        <box size=" ${L3 - MotorOffset*2} ${LinkWidth} ${LinkHeight}"/>
+      </geometry>
+    </collision>
+    <collision>
+      <origin xyz="${L3 - 0.01} 0 ${d3}" rpy="0 0 0"/>
+      <geometry>
+        <box size=" ${0.045} ${MotorLength} ${MotorWidth*2 - 0.005}"/>
       </geometry>
     </collision>
@@ -145,5 +172,5 @@
       <origin xyz="0 0 0" rpy="0 ${M_pi/2} 0"/>
       <geometry>
-        <mesh filename="package://crustcrawler_description/meshes/Link3.STL"/> <!--<box size="${L3} ${LinkWidth} ${LinkWidth} "/> -->
+        <mesh filename="package://crustcrawler_description/meshes/Link3.STL"/>
       </geometry>
     </visual>
@@ -176,5 +203,5 @@
   <link name="gripper_left">
     <collision>
-      <origin xyz="0 0 0" rpy="0 0 0.1"/>
+      <origin xyz="0 0 5" rpy="0 0 0.1"/>
       <geometry>
   <box size=" ${LinkWidth} ${LinkWidth} ${LinkWidth}"/>
@@ -199,5 +226,5 @@
   <link name="gripper_right">
     <collision>
-      <origin xyz="0 0 0" rpy="0 0 0"/>
+      <origin xyz="0 0 5" rpy="0 0 0"/>
       <geometry>
   <box size=" ${LinkWidth} ${LinkWidth} ${LinkWidth}"/>
