Commit message: added inertia

File: src/crustcrawler_description/urdf/crustcrawler.xacro (robot description, xacro)
@@ -69,7 +69,7 @@
     </inertial>
   </link>
-  <joint name="joint1" type="revolute">
-    <axis xyz="0 0 1"/>
-    <limit effort="1000.0" lower="${-M_pi}" upper="${M_pi}" velocity="0.5"/>
+  <joint name="joint1" type="continuous">
+    <axis xyz="0 0 1"/>
+    <!--limit effort="1000.0" lower="${-M_pi}" upper="${M_pi}" velocity="0.5"/ -->
     <parent link="base"/>
     <child link="link1"/>
@@ -105,13 +105,12 @@
       <mass value="${m1}"/>
       <inertia
-    	  ixx="1.0" ixy="0.0" ixz="0.0"
-    	  iyy="1.0" iyz="0.0"
-    	  izz="1.0"/>
-    </inertial>
-  </link>
-  <joint name="joint2" type="revolute">
+    	  ixx="0.08410695" ixy="-0.00213140" ixz="-0.00685242"
+    	  iyy="0.11802166" iyz="0.00036003"
+    	  izz="0.11395469"/>
+    </inertial>
+  </link>
+  <joint name="joint2" type="continuous">
     <origin xyz="0 0 ${L1}" rpy="${M_pi / 2} 0 0"/>
     <axis xyz="0 0 1"/>
-    <limit effort="1000.0" lower="${-M_pi/4}" upper="${M_pi*5/4}" velocity="0.5"/>
     <parent link="link1"/>
     <child link="link2"/>
@@ -142,12 +141,11 @@
       <mass value="${m2}"/>
       <inertia
-	  ixx="1.0" ixy="0.0" ixz="0.0"
-	  iyy="1.0" iyz="0.0"
-	  izz="1.0"/>
-    </inertial>
-  </link>
-  <joint name="joint3" type="revolute">
-    <axis xyz="0 0 1"/>
-    <limit effort="1000.0" lower="${-M_pi*3/4}" upper="${M_pi*3/4}" velocity="0.5"/>
+	  ixx="0.63396931" ixy="-0.01273805" ixz="-0.01536619"
+	  iyy="0.01536619" iyz="0.26329519"
+	  izz="0.44043802"/>
+    </inertial>
+  </link>
+  <joint name="joint3" type="continuous">
+    <axis xyz="0 0 1"/>
     <parent link="link2"/>
     <child link="link3"/>
@@ -179,12 +177,11 @@
       <mass value="${m3}"/>
       <inertia
-    ixx="1.0" ixy="0.0" ixz="0.0"
-    iyy="1.0" iyz="0.0"
-    izz="1.0"/>
-    </inertial>
-  </link>
-  <joint name="joint4" type="revolute">
-    <axis xyz="0 0 1"/>
-    <limit effort="1000.0" lower="${-M_pi*3/4}" upper="${M_pi*3/4}" velocity="0.5"/>
+    ixx="0.25596532" ixy="0.00155757" ixz="-0.01187757"
+    iyy="0.32784813" iyz="-0.02519485"
+    izz="0.02519485"/>
+    </inertial>
+  </link>
+  <joint name="joint4" type="continuous">
+    <axis xyz="0 0 1"/>
     <parent link="link3"/>
     <child link="gripper_left"/>
@@ -192,7 +189,6 @@
     <dynamics damping="0.7"/>
   </joint>
-  <joint name="joint5" type="revolute">
-    <axis xyz="0 0 1"/>
-    <limit effort="1000.0" lower="${-M_pi*3/4}" upper="${M_pi*3/4}" velocity="0.5"/>
+  <joint name="joint5" type="continuous">
+    <axis xyz="0 0 1"/>
     <parent link="link3"/>
     <child link="gripper_right"/>
@@ -203,7 +199,7 @@
   <link name="gripper_left">
     <collision>
-      <origin xyz="0 0 5" rpy="0 0 0.1"/>
-      <geometry>
-  <box size=" ${LinkWidth} ${LinkWidth} ${LinkWidth}"/>
+      <origin xyz="0 0 1" rpy="0 0 0"/>
+      <geometry>
+        <box size=" ${LinkWidth} ${LinkWidth} ${LinkWidth}"/>
       </geometry>
     </collision>
@@ -218,7 +214,7 @@
       <mass value="0.001"/>
       <inertia
-    ixx="1.0" ixy="0.0" ixz="0.0"
-    iyy="1.0" iyz="0.0"
-    izz="1.0"/>
+    ixx="0.0" ixy="0.0" ixz="0.0"
+    iyy="0.0" iyz="0.0"
+    izz="0.0"/>
     </inertial>
   </link>
@@ -226,7 +222,7 @@
   <link name="gripper_right">
     <collision>
-      <origin xyz="0 0 5" rpy="0 0 0"/>
-      <geometry>
-  <box size=" ${LinkWidth} ${LinkWidth} ${LinkWidth}"/>
+      <origin xyz="0 0 1" rpy="0 0 0"/>
+      <geometry>
+        <box size=" ${LinkWidth} ${LinkWidth} ${LinkWidth}"/>
       </geometry>
     </collision>
@@ -241,7 +237,7 @@
       <mass value="0.001"/>
       <inertia
-    ixx="1.0" ixy="0.0" ixz="0.0"
-    iyy="1.0" iyz="0.0"
-    izz="1.0"/>
+    ixx="0.0" ixy="0.0" ixz="0.0"
+    iyy="0.0" iyz="0.0"
+    izz="0.0"/>
     </inertial>
   </link>

Commit message: cleanup

File: src/crustcrawler_description/urdf/crustcrawler.xacro (robot description, xacro)
@@ -77,14 +77,4 @@
     <dynamics damping="0.7"/>
   </joint>
-  <transmission name="tran1">
-    <type>transmission_interface/SimpleTransmission</type>
-    <joint name="joint1">
-      <hardwareInterface>hardware_interface/EffortJointInterface</hardwareInterface>
-    </joint>
-    <actuator name="motor1">
-      <hardwareInterface>hardware_interface/EffortJointInterface</hardwareInterface>
-      <mechanicalReduction>1</mechanicalReduction>
-    </actuator>
-  </transmission>
   <!-- link 1 -->
   <link name="link1">
